Commit message: package:// syntax changed in URDF

File: urdf/draco3.urdf (robot description, URDF)
Before this commit: robot draco_3, 48 links, 47 joints
Links:
- link l_ankle_fe_link: geometry visual mesh filename=package://draco3_description/meshes/l_ankle_fe_link.stl
- link l_ankle_ie_link: geometry collision box size=0.25 0.15 0.0591; visual mesh filename=package://draco3_description/meshes/l_ankle_ie_link.stl
- link l_elbow_fe_link: geometry visual mesh filename=package://draco3_description/meshes/l_elbow_fe_link.stl
- link l_hip_aa_link: geometry visual mesh filename=package://draco3_description/meshes/l_hip_aa_link.stl
- link l_hip_fe_link: geometry visual mesh filename=package://draco3_description/meshes/l_hip_fe_link3.obj
- link l_hip_ie_link: geometry visual mesh filename=package://draco3_description/meshes/l_hip_ie_link.stl
- link l_knee_adj_link: geometry visual mesh filename=package://draco3_description/meshes/l_knee_adj_link.stl
- link l_knee_fe_ld: geometry visual mesh filename=package://draco3_description/meshes/l_knee_fe_ld3.obj
- link l_knee_fe_lp: geometry visual mesh filename=package://draco3_description/meshes/l_knee_fe_lp.stl
- link l_sake_gripper_link: geometry visual mesh filename=package://draco3_description/meshes/l_sake_gripper_mount.stl
- link l_shoulder_aa_link: geometry visual mesh filename=package://draco3_description/meshes/l_shoulder_aa_link.stl
- link l_shoulder_fe_link: geometry visual mesh filename=package://draco3_description/meshes/l_shoulder_fe_link.stl
- link l_shoulder_ie_link: geometry visual mesh filename=package://draco3_description/meshes/l_shoulder_ie_link3.obj
- link l_wrist_ps_link: geometry visual mesh filename=package://draco3_description/meshes/l_wrist_ps_link.stl
- link left_ezgripper_finger_L1_1: geometry visual mesh filename=package://draco3_description/meshes/ezgripper_gen2/SAKE_Fin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
- link left_ezgripper_finger_L1_2: geometry visual mesh filename=package://draco3_description/meshes/ezgripper_gen2/SAKE_Fin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
- link left_ezgripper_finger_L2_1: geometry collision mesh filename=package://draco3_description/meshes/ezgripper_gen2/SAKE_Fin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; visual mesh filename=package://draco3_description/meshes/ezgripper_gen2/SAKE_Fin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
- link left_ezgripper_finger_L2_2: geometry collision mesh filename=package://draco3_description/meshes/ezgripper_gen2/SAKE_Fin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; visual mesh filename=package://draco3_description/meshes/ezgripper_gen2/SAKE_Fin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
- link left_ezgripper_palm_link: geometry visual mesh filename=package://draco3_description/meshes/ezgripper_gen2/SAKE_Pal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
- link neck_pitch_link: geometry visual mesh filename=package://draco3_description/meshes/neck_pitch_link3.obj
- link r_ankle_fe_link: geometry visual mesh filename=package://draco3_description/meshes/r_ankle_fe_link.stl
- link r_ankle_ie_link: geometry collision box size=0.25 0.15 0.0591; visual mesh filename=package://draco3_description/meshes/r_ankle_ie_link.stl
- link r_elbow_fe_link: geometry visual mesh filename=package://draco3_description/meshes/r_elbow_fe_link.stl
- link r_hip_aa_link: geometry visual mesh filename=package://draco3_description/meshes/r_hip_aa_link.stl
- link r_hip_fe_link: geometry visual mesh filename=package://draco3_description/meshes/r_hip_fe_link3.obj
- link r_hip_ie_link: geometry visual mesh filename=package://draco3_description/meshes/r_hip_ie_link.stl
- link r_knee_adj_link: geometry visual mesh filename=package://draco3_description/meshes/r_knee_adj_link.stl
- link r_knee_fe_ld: geometry visual mesh filename=package://draco3_description/meshes/r_knee_fe_ld3.obj
- link r_knee_fe_lp: geometry visual mesh filename=package://draco3_description/meshes/r_knee_fe_lp.stl
- link r_sake_gripper_link: geometry visual mesh filename=package://draco3_description/meshes/r_sake_gripper_mount.stl
- link r_shoulder_aa_link: geometry visual mesh filename=package://draco3_description/meshes/r_shoulder_aa_link.stl
- link r_shoulder_fe_link: geometry visual mesh filename=package://draco3_description/meshes/r_shoulder_fe_link.stl
- link r_shoulder_ie_link: geometry visual mesh filename=package://draco3_description/meshes/r_shoulder_ie_link3.obj
- link r_wrist_ps_link: geometry visual mesh filename=package://draco3_description/meshes/r_wrist_ps_link.stl
- link right_ezgripper_finger_L1_1: geometry visual mesh filename=package://draco3_description/meshes/ezgripper_gen2/SAKE_Fin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
- link right_ezgripper_finger_L1_2: geometry visual mesh filename=package://draco3_description/meshes/ezgripper_gen2/SAKE_Fin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
- link right_ezgripper_finger_L2_1: geometry collision mesh filename=package://draco3_description/meshes/ezgripper_gen2/SAKE_Fin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; visual mesh filename=package://draco3_description/meshes/ezgripper_gen2/SAKE_Fin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
- link right_ezgripper_finger_L2_2: geometry collision mesh filename=package://draco3_description/meshes/ezgripper_gen2/SAKE_Fin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; visual mesh filename=package://draco3_description/meshes/ezgripper_gen2/SAKE_Fin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
- link right_ezgripper_palm_link: geometry visual mesh filename=package://draco3_description/meshes/ezgripper_gen2/SAKE_Pal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
- link torso_link: geometry visual mesh filename=package://draco3_description/meshes/torso_link3.obj
